File: hardware/Solderable_Breadboard_Large.sch (EAGLE design)
At the start: 161 parts

Commit message: Renamed files to match product name, and updates from reviewing protos.
Parts:
- removed JP150, JP151, JP152, JP153, JP65, JP66, JP67, JP68: M01SMDNS, SparkFun-Connectors:M01SMDNS
- added JG1, JG2, JG3, JG4, JG5, JG6: M021X02_NO_SILK, SparkFun-Connectors:M021X02_NO_SILK
- added TIE+1, TIE+2, TIE-1, TIE-2: M01SMDNS, SparkFun-Connectors:M01SMDNS
Connections:
- removed net N$65: JP65.1, S2.P$1
- removed net N$66: JP66.1, S1.P$1
- new net N$1: JG1.2, S1.P$1
- new net N$2: JG2.2, S2.P$1
- net GND: now also JG1.1, JG2.1, JG3.2, JG4.2, JG5.2, JG6.1; no longer JP150.1, JP151.1, JP152.1, JP153.1
- net N$67: now also JG3.1; no longer JP67.1
- net N$68: now also JG4.1; no longer JP68.1
- net V+BOT: now also TIE+2.1
- net V+TOP: now also TIE+1.1
- net V-BOT: now also JG6.2, TIE-2.1
- net V-TOP: now also JG5.1, TIE-1.1
Other:
- note added: "This board offers several strapping options: -JG1, JG2, JG3, JG4 allow for the mounting holes to be connected to ground, if you want to ground to a metal enclosure. -JG5, JG6 tie the V- rails to ground, so V- can be used interchangably with ground. This is useful for digital logic circuits when only require ground and VCC. -TIE+1, TIE-1, TIE+2, TIE-2 allow the rais at the top of the board to be t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"
- moved on the sheet: JP147, JP149, S1, S2, S3, S4
